Commit message: added rviz launcher

File: src/maze_robot/urdf/robot.xacro (robot description, xacro)
@@ -4,5 +4,5 @@
   <!-- Mathematical constant -->
   <!-- ===================== -->
-  <xacro:property name="pi" value="3.14159265"/>
+  <xacro:property name="pi_const" value="3.14159265"/>
   <!-- ===================== -->
   <!-- Robot body dimensions -->
@@ -44,7 +44,7 @@
                   value="${chassis_density * chassis_length * chassis_height * chassis_width}"/>
   <xacro:property name="wheel_mass"
-                  value="${wheel_density * pi * wheel_radius * wheel_radius * wheel_width}"/>
+                  value="${wheel_density * pi_const * wheel_radius * wheel_radius * wheel_width}"/>
   <xacro:property name="caster_mass"
-                  value="${caster_density * (4.0/3.0) * pi * wheel_radius * wheel_radius * wheel_radius}"/>
+                  value="${caster_density * (4.0/3.0) * pi_const * wheel_radius * wheel_radius * wheel_radius}"/>
   <!-- ===================== -->
   <!-- Inertia calculations -->

Commit message: added lidar and camera

File: src/maze_robot/urdf/robot.xacro (robot description, xacro)
@@ -125,4 +125,60 @@
   </link>
   <!-- ===================== -->
+<!-- LiDAR joint -->
+<!-- ===================== -->
+<joint name="lidar_joint" type="fixed">
+  <!-- Mount LiDAR on top of the chassis -->
+  <origin xyz="0 0 ${chassis_z_offset + wheel_radius}" rpy="0 0 0"/>
+  <parent link="body_link"/>
+  <child link="lidar_link"/>
+</joint>
+<!-- ===================== -->
+<!-- LiDAR link -->
+<!-- ===================== -->
+<link name="lidar_link">
+  <visual>
+    <origin xyz="0 0 0.05" rpy="0 0 0"/>
+    <geometry>
+      <cylinder length="0.1" radius="0.1"/>
+    </geometry>
+    <material name="lidar_black">
+      <color rgba="0 0 0 1"/>
+    </material>
+  </visual>
+  <collision>
+    <origin xyz="0 0 0.05" rpy="0 0 0"/>
+    <geometry>
+      <cylinder length="0.1" radius="0.1"/>
+    </geometry>
+  </collision>
+  <inertial>
+    <!-- Very small mass to avoid affecting dynamics -->
+    <mass value="1e-6"/>
+    <origin xyz="0 0 0" rpy="0 0 0"/>
+    <inertia
+      ixx="1e-6" ixy="0" ixz="0"
+      iyy="1e-6" iyz="0"
+      izz="1e-6"/>
+  </inertial>
+</link>
+  <!-- ===================== -->
+  <!-- Camera sensor -->
+  <!-- ===================== -->
+  <joint name="camera_joint" type="fixed">
+    <parent link="body_link"/>
+    <child link="camera_link"/>
+    <origin xyz="0.52 0 0.4" rpy="0 0 0"/>
+  </joint>
+  <link name="camera_link">
+    <visual>
+      <geometry>
+        <box size="0.05 0.05 0.05"/>
+      </geometry>
+      <material name="camera_blue">
+        <color rgba="0 0 1 1"/>
+      </material>
+    </visual>
+  </link>
+  <!-- ===================== -->
   <!-- Left wheel -->
   <!-- ===================== -->

Commit message: fixed lidar scan arc visibilty problem

File: src/maze_robot/urdf/robot.xacro (robot description, xacro)
@@ -112,6 +112,6 @@
         <box size="${chassis_length} ${chassis_width} ${chassis_height}"/>
       </geometry>
-      <material name="chassis_red">
-        <color rgba="1 0 0 1"/>
+      <material name="chassis_blue">
+        <color rgba="0 0.6 0.6 1"/>
       </material>
     </visual>
@@ -142,6 +142,6 @@
       <cylinder length="0.1" radius="0.1"/>
     </geometry>
-    <material name="lidar_black">
-      <color rgba="0 0 0 1"/>
+    <material name="lidar_purple">
+      <color rgba="0.3 0 0.5 1"/>
     </material>
   </visual>
@@ -173,8 +173,8 @@
     <visual>
       <geometry>
-        <box size="0.05 0.05 0.05"/>
+        <box size="0.07 0.07 0.07"/>
       </geometry>
       <material name="camera_blue">
-        <color rgba="0 0 1 1"/>
+        <color rgba="0 0 0 1"/>
       </material>
     </visual>
@@ -197,6 +197,6 @@
         <cylinder radius="${wheel_radius}" length="${wheel_width}"/>
       </geometry>
-      <material name="wheel_yellow">
-        <color rgba="1 1 0 1"/>
+      <material name="wheel_grey">
+        <color rgba="0.8 0.8 0.8 1"/>
       </material>
     </visual>
@@ -226,6 +226,6 @@
         <cylinder radius="${wheel_radius}" length="${wheel_width}"/>
       </geometry>
-      <material name="wheel_yellow">
-        <color rgba="1 1 0 1"/>
+      <material name="wheel_grey">
+        <color rgba="0.8 0.8 0.8 1"/>
       </material>
     </visual>

Commit message: Added code block to launch rviz map without erro

File: src/maze_robot/urdf/robot.xacro (robot description, xacro)
@@ -98,9 +98,21 @@
   <!-- Base footprint -->
   <!-- ===================== -->
+<link name="base_link"/>
   <link name="base_footprint"/>
+  <joint name="base_link_to_footprint" type="fixed">
+    <parent link="base_link"/>
+    <child link="base_footprint"/>
+    <origin xyz="0 0 0" rpy="0 0 0"/>
+  </joint>
   <joint name="base_to_chassis" type="fixed">
-    <parent link="base_footprint"/>
+    <parent link="base_link"/>
     <child link="body_link"/>
-  </joint>
+    <origin xyz="0 0 0" rpy="0 0 0"/>
+  </joint>
+  <!--<link name="base_footprint"/> -->
+  <!--<joint name="base_to_chassis" type="fixed"> -->
+  <!--  <parent link="base_footprint"/>-->
+  <!--  <child link="body_link"/>-->
+  <!--</joint>-->
   <!-- ===================== -->
   <!-- Chassis link -->
